Commit message: delete: 移除旧版宇树L6连接装配文件

File: updf_Robotic/unitree_l6_link_001/urdf/unitree_l6_link_001.urdf (robot description, URDF)
Before this commit: robot 宇树L6连接001.SLDASM, 1 links, 0 joints
Links:
- link base_link: mass 0.0388754856381894 -> 0.040989831193917; geometry collision mesh filename=package://unitree_l6_link_001/meshes/base_link.STL; visual mesh filename=package://unitree_l6_link_001/meshes/base_link.STL
