Commit message: fix: Active_Vision_Platform_001 同步修正Empty_Link1相对位姿，维持装配相对关系1. base_link网格归零后，同步平移Empty_Link1坐标，保证底座与云台原有装配间隙不变2. Empty_Link2相对于Empty_Link1位姿保持原样，完整保留连杆层级结构3. URDF、MuJoCo xml惯性原点、连杆pos全部统一至世界原点，仿真无模型漂移、零件分离问题

File: updf_Robotic/Active_Vision_Platform_001/urdf/Active_Vision_Platform.urdf (robot description, URDF)
Before this commit: robot Active_Vision_Platform, 3 links, 2 joints
Joints:
- joint joint1: origin xyz=0.31194 -0.10063 -0.3345 rpy=3.1351 0.967 -1.5786 -> xyz=-0.009349 -0.025641 -0.013045 rpy=3.1351 0.967 -1.5786
